Commit message: update urdf

File: urdf/atom01.urdf (robot description, URDF)
Before this commit: robot atom01urdf, 24 links, 23 joints
Links:
- link base_link: mass 5.38006123 -> 5.50170905 
- link left_ankle_roll_link: mass 0.32034036  -> 0.30640039 
- link left_arm_pitch_link: mass 0.48107005 -> 0.47050957
- link left_arm_roll_link: mass 0.10569114 -> 0.09168685
- link left_arm_yaw_link: mass 1.15030164 -> 1.15324429
- link left_elbow_pitch_link: mass 0.10324612 -> 0.09168685
- link left_elbow_yaw_link: mass 0.67956658 -> 0.68145673 
- link left_thigh_pitch_link: mass 2.34679679 ->  2.34227381
- link left_thigh_roll_link: mass 1.71072574 -> 1.71445955  
- link left_thigh_yaw_link: mass 1.70245957 -> 1.68565743 
- link right_ankle_roll_link: mass 0.32034036 ->  0.30640039
- link right_arm_pitch_link: mass 0.48107005 -> 0.47178757
- link right_arm_roll_link: mass 0.10324612 -> 0.09168685
- link right_arm_yaw_link: mass 1.14935657 -> 1.15196629
- link right_elbow_pitch_link: mass 0.10569114 -> 0.09168685
- link right_knee_link: mass 1.79036871 ->  1.79131378
- link right_thigh_pitch_link: mass 2.34679679 -> 2.34600762
- link torso_link: mass 7.65615208 -> 7.70005232 

Commit message: update xml&urdf

File: urdf/atom01.urdf (robot description, URDF)
Before this commit: robot atom01urdf, 24 links, 23 joints
Links:
- link base_link: mass 5.50170905  -> 5.38006123
- link left_arm_pitch_link: mass 0.47050957 -> 0.47178757
- link left_elbow_yaw_link: mass 0.68145673  -> 0.68145673
- link left_knee_link: mass 1.79036871  -> 1.79036871
- link left_thigh_pitch_link: mass  2.34227381 -> 2.34600762
- link left_thigh_roll_link: mass 1.71445955   -> 1.71632646
- link left_thigh_yaw_link: mass 1.68565743  -> 1.68866185
- link right_arm_yaw_link: mass 1.15196629 -> 1.15324429
- link right_knee_link: mass  1.79131378 -> 1.79036871
- link right_thigh_roll_link: mass 1.71072574 -> 1.71632646

Commit message: update limit

File: urdf/atom01.urdf (robot description, URDF)
Before this commit: robot atom01urdf, 24 links, 23 joints
Joints:
- joint left_arm_pitch_joint: limit lower=-1.57 upper=1.57 effort=18 velocity=3.7692 -> lower=-3.14 upper=1.57 effort=18 velocity=3.7692
- joint left_arm_roll_joint: limit lower=-0.25 upper=1 effort=18 velocity=3.7692 -> lower=-0.25 upper=3.14 effort=18 velocity=3.7692
- joint right_arm_pitch_joint: limit lower=-1.57 upper=1.57 effort=18 velocity=3.7692 -> lower=-3.14 upper=1.57 effort=18 velocity=3.7692
- joint right_arm_roll_joint: limit lower=-1 upper=0.25 effort=18 velocity=3.7692 -> lower=-3.14 upper=0.25 effort=18 velocity=3.7692

Commit message: update limits

File: urdf/atom01.urdf (robot description, URDF)
Before this commit: robot atom01urdf, 24 links, 23 joints
Joints:
- joint left_thigh_pitch_joint: limit lower=-1 upper=1 effort=80 velocity=10.47 -> lower=-1.57 upper=1.57 effort=80 velocity=10.47
- joint right_thigh_pitch_joint: limit lower=-1 upper=1 effort=80 velocity=10.47 -> lower=-1.57 upper=1.57 effort=80 velocity=10.47
